Commit message: [RS-177] Update arm model to full version

File: catkin_ws/src/arm_description/urdf/arm.URDF (robot description, URDF)
Before this commit: robot Assem, 3 links, 2 joints
Links:
- removed link baseyaw
- added link arm_base, mass 1.07263545959926; collision mesh filename=package://arm_description/meshes/arm_base.STL; visual mesh filename=package://arm_description/meshes/arm_base.STL
- added link diff1, mass 0.22290258094587; collision mesh filename=package://arm_description/meshes/diff1.STL; visual mesh filename=package://arm_description/meshes/diff1.STL
- added link diff2, mass 0.109394214433751; collision mesh filename=package://arm_description/meshes/diff2.STL; visual mesh filename=package://arm_description/meshes/diff2.STL
- added link end_effector, mass 0.18801084998517; collision mesh filename=package://arm_description/meshes/end_effector.STL; visual mesh filename=package://arm_description/meshes/end_effector.STL
- added link finger1, mass 0.0227611478993928; collision mesh filename=package://arm_description/meshes/finger1.STL; visual mesh filename=package://arm_description/meshes/finger1.STL
- added link finger2, mass 0.0227611430860343; collision mesh filename=package://arm_description/meshes/finger2.STL; visual mesh filename=package://arm_description/meshes/finger2.STL
- added link link2, mass 0.580638766374297; collision mesh filename=package://arm_description/meshes/link2.STL; visual mesh filename=package://arm_description/meshes/link2.STL
- link link1: mass 1.36312424561291 -> 1.36045203504809
Joints:
- removed joint pitch1
- removed joint yaw1
- added joint base_pitch: type continuous, parent arm_base, child link1, origin xyz=0 0.0750951 0 rpy=0.442957283043391 6.10622663543836E-16 2.85064834697979E-16, axis -1 0 0
- added joint base_yaw: type continuous, parent base_link, child arm_base, origin xyz=0 0 0.00634999999999998 rpy=1.5707963267949 -2.3371962784201E-17 -1.8628998344518, axis 0 -1 0
- added joint pitch2: type continuous, parent link1, child diff1, origin xyz=0 0.452768804137388 -0.0635 rpy=0.152152878773275 1.27675647831893E-15 3.14159265358979, axis 1 0 0
- added joint pitch3: type continuous, parent link2, child diff2, origin xyz=0 0.432430108178054 0 rpy=3.12735368407058 -1.38777878078145E-16 -6.66133814775094E-16, axis -1 0 0
- added joint roll1: type continuous, parent diff1, child link2, origin xyz=0 0 0.00906290817805414 rpy=-1.5707963267949 4.9960036108132E-16 -3.02066843525624, axis 0 -1 0
- added joint roll2: type continuous, parent diff2, child end_effector, origin xyz=0 0 -0.0768495238393263 rpy=-1.57079632679489 3.08086889333481E-15 0.379261683076635, axis 0 -1 0
- added joint slide_finger1: type prismatic, parent end_effector, child finger1, origin xyz=0.00160020 0.038949 0 rpy=0 1.5708 0, axis 0 0 1, limit lower=0.0 upper=0.0473958 effort=0 velocity=0
- added joint slide_finger2: type prismatic, parent end_effector, child finger2, origin xyz=-0.00160020 0.038949 0 rpy=0 -1.5708 0, axis 0 0 1, limit lower=0.0 upper=0.0473958 effort=0 velocity=0

Commit message: [RS-177] Make finger of the end effector move symmetrically

File: catkin_ws/src/arm_description/urdf/arm.URDF (robot description, URDF)
Before this commit: robot arm_description, 9 links, 8 joints
Joints:
- joint slide_finger2: mimic (none) -> joint=slide_finger1
