Commit message: Add ros_control controllers for the arm and a gazebo world

File: catkin_ws/src/arm_description/urdf/arm.urdf (robot description, URDF)
Before this commit: robot arm_description, 9 links, 8 joints
Joints:
- joint slide_finger1: limit lower=0.0 upper=0.0473958 effort=0 velocity=0 -> lower=0.0 upper=0.0473958 effort=1000000 velocity=1000000
- joint slide_finger2: limit lower=0.0 upper=0.0473958 effort=0 velocity=0 -> lower=0.0 upper=0.0473958 effort=1000000 velocity=1000000

Commit message: Tune PID values of controllers for the arm

File: catkin_ws/src/arm_description/urdf/arm.urdf (robot description, URDF)
Before this commit: robot arm, 9 links, 8 joints
Links:
- added link world
Joints:
- added joint world_fix: type fixed, parent world, child base_link, origin xyz=0 0 0 rpy=0 0 0
- joint base_pitch: limit (none) -> effort=200.0 velocity=2.0
- joint base_yaw: limit (none) -> effort=200.0 velocity=2.0
- joint pitch2: limit (none) -> effort=200.0 velocity=2.0
- joint pitch3: limit (none) -> effort=200.0 velocity=2.0
- joint roll1: limit (none) -> effort=200.0 velocity=0.5
- joint roll2: limit (none) -> effort=200.0 velocity=0.5
- joint slide_finger1: limit lower=0.0 upper=0.0473958 effort=1000000 velocity=1000000 -> lower=0.0 upper=0.0473958 effort=200.0 velocity=2.0
- joint slide_finger2: limit lower=0.0 upper=0.0473958 effort=1000000 velocity=1000000 -> lower=0.0 upper=0.0473958 effort=200.0 velocity=2.0; mimic joint=slide_finger1 -> (none)

Commit message: Add pass-through action servers linking MoveIt! and ros_control (#198)

File: catkin_ws/src/arm_description/urdf/arm.urdf (robot description, URDF)
Before this commit: robot arm, 10 links, 9 joints
Joints:
- joint slide_finger1: type prismatic -> fixed
- joint slide_finger2: type prismatic -> fixed

Commit message: Clarify arm joint names for Moveit (#225)

File: catkin_ws/src/arm_description/urdf/arm.urdf (robot description, URDF)
Before this commit: robot arm, 10 links, 9 joints
Joints:
- removed joint pitch2
- removed joint pitch3
- removed joint roll1
- removed joint roll2
- added joint elbow_pitch: type continuous, parent link1, child diff1, origin xyz=0 0.452768804137388 -0.0635 rpy=0.152152878773275 1.27675647831893E-15 3.14159265358979, axis 1 0 0, limit effort=200.0 velocity=2.0
- added joint elbow_roll: type continuous, parent diff1, child link2, origin xyz=0 0 0.00906290817805414 rpy=-1.5707963267949 4.9960036108132E-16 -3.02066843525624, axis 0 -1 0, limit effort=200.0 velocity=0.5
- added joint wrist_pitch: type continuous, parent link2, child diff2, origin xyz=0 0.432430108178054 0 rpy=3.12735368407058 -1.38777878078145E-16 -6.66133814775094E-16, axis -1 0 0, limit effort=200.0 velocity=2.0
- added joint wrist_roll: type continuous, parent diff2, child end_effector, origin xyz=0 0 -0.0768495238393263 rpy=-1.57079632679489 3.08086889333481E-15 0.379261683076635, axis 0 -1 0, limit effort=200.0 velocity=0.5

Commit message: Add bounding boxes to the arm joints (#224)

File: catkin_ws/src/arm_description/urdf/arm.urdf (robot description, URDF)
Before this commit: robot arm, 10 links, 9 joints
Links:
- link arm_base: geometry collision mesh filename=package://arm_description/meshes/obbs/arm_base_obb.STL; visual mesh filename=package://arm_description/meshes/arm_base.STL
- link base_link: geometry collision mesh filename=package://arm_description/meshes/obbs/base_link_obb.STL; visual mesh filename=package://arm_description/meshes/base_link.STL
- link diff1: geometry collision mesh filename=package://arm_description/meshes/obbs/diff1_obb.STL; visual mesh filename=package://arm_description/meshes/diff1.STL
- link diff2: geometry collision mesh filename=package://arm_description/meshes/obbs/diff2_obb.STL; visual mesh filename=package://arm_description/meshes/diff2.STL
- link end_effector: geometry collision mesh filename=package://arm_description/meshes/obbs/end_effector_obb.STL; visual mesh filename=package://arm_description/meshes/end_effector.STL
- link finger1: geometry collision mesh filename=package://arm_description/meshes/obbs/finger1_obb.STL; visual mesh filename=package://arm_description/meshes/finger1.STL
- link finger2: geometry collision mesh filename=package://arm_description/meshes/obbs/finger2_obb.STL; visual mesh filename=package://arm_description/meshes/finger2.STL
- link link1: geometry collision mesh filename=package://arm_description/meshes/obbs/link1_obb.STL; visual mesh filename=package://arm_description/meshes/link1.STL
- link link2: geometry collision mesh filename=package://arm_description/meshes/obbs/link2_obb.STL; visual mesh filename=package://arm_description/meshes/link2.STL
